Commit message: feat: change serialization to new one, write own sensor converter, changed time to microsec, add error handler
Signed-off-by: Maciej Krupka <maciej.p.krupka@student.put.poznan.pl>

File: urdf/av21.urdf (robot description, URDF)
Before this commit: robot AV21, 22 links, 21 joints
Links:
- added link camera_front_link
Joints:
- added joint camera_front_link_joint: type fixed, parent rear_axle_middle, child camera_front_link, origin xyz=2.184 0 0.422
